File: ctrl_main/ctrl_main.sch (KiCad schematic (older format))
At the start: 19 parts, among them IC1 SN74HC125N, J1 B2B-XH-A(LF)(SN), J2 B2B-XH-A(LF)(SN), J3 B2B-XH-A(LF)(SN), P11 CONN_01X03, P12 CONN_01X03, P4 CONN_01X04, P5 CONN_01X04, P6 CONN_01X04, P7 CONN_01X04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

Commit message: 測定系との通信コネクタを4p->3pに変更（5Vを削除）
Parts:
- P1: renamed from P?; footprint (none) -> Pin_Headers:Pin_Header_Straight_1x03_Pitch1.27mm
Connections:
- net at Q2.2 (C), R4.1: now also IC1.13 (4~OE); no longer IC1.10 (3~OE)
- net at P8.2 (P2), R2.2: now also IC1.10 (3~OE); no longer IC1.13 (4~OE)
Changed lines of the file:
@@
 Wire Wire Line
 	5450 1350 5450 4650
-Wire Wire Line
-	7150 4450 7550 4450
-Wire Wire Line
-	7550 4450 7550 3100
-Wire Wire Line
-	6350 4650 6350 3700
-Wire Wire Line
-	6350 3700 7250 3700
-Wire Wire Line
-	7250 3700 7250 3100
 Connection ~ 6350 4650
 Text GLabel 7150 4100 1    60   Input ~ 0
@@
 $EndComp
 $Comp
-L CONN_01X03 P?
+L CONN_01X03 P1
 U 1 1 5909467D
 P 6250 5350
-F 0 "P?" H 6250 5550 50  0000 C CNN
+F 0 "P1" H 6250 5550 50  0000 C CNN
 F 1 "CONN_01X03" V 6350 5350 50  0000 C CNN
-F 2 "" H 6250 5350 50  0000 C CNN
+F 2 "Pin_Headers:Pin_Header_Straight_1x03_Pitch1.27mm" H 6250 5350 50  0001 C CNN
 F 3 "" H 6250 5350 50  0000 C CNN
 	1    6250 5350
@@
 Wire Wire Line
 	6150 2500 6150 5150
+Wire Wire Line
+	7250 3100 7250 4450
+Wire Wire Line
+	7250 4450 7150 4450
+Wire Wire Line
+	6350 4650 6350 3750
+Wire Wire Line
+	6350 3750 7550 3750
+Wire Wire Line
+	7550 3750 7550 3100
 $EndSCHEMATC
