File: pitch_sensor/pitch_sensor.sch (KiCad schematic (older format))
At the start: 27 parts, among them IC1 DEV-11114, P1 CONN_01X21

Commit message: mod pitch_sensor
Parts:
- D1, R1: footprint (none) -> Air_Coils_SML_NEOSID:Neosid_Air-Coil_SML_1turn_HDM0131A
- D10, R9: footprint (none) -> Air_Coils_SML_NEOSID:Neosid_Air-Coil_SML_5turn_HDM0531A
- D11, R10: footprint (none) -> Air_Coils_SML_NEOSID:Neosid_Air-Coil_SML_6-10turn_HAM0631A-HAM1031A
- D12, R11: footprint (none) -> Air_Coils_SML_NEOSID:Neosid_Air-Coil_SML_6-10turn_HDM0431A-HDM1031A
- D2, D3, R2, R3: footprint (none) -> Air_Coils_SML_NEOSID:Neosid_Air-Coil_SML_2turn_HAM0231A
- D4, R4, R5: footprint (none) -> Air_Coils_SML_NEOSID:Neosid_Air-Coil_SML_2turn_HDM0231A
- D5, R6: footprint (none) -> Air_Coils_SML_NEOSID:Neosid_Air-Coil_SML_3turn_HAM0331A
- D6, R7: footprint (none) -> Air_Coils_SML_NEOSID:Neosid_Air-Coil_SML_3turn_HDM0331A
- D7: footprint (none) -> Air_Coils_SML_NEOSID:Neosid_Air-Coil_SML_4turn_HAM0431A
- D8: footprint (none) -> Air_Coils_SML_NEOSID:Neosid_Air-Coil_SML_4turn_HDM0431A
- D9, R8: footprint (none) -> Air_Coils_SML_NEOSID:Neosid_Air-Coil_SML_5turn_HAM0531A
- R12: footprint (none) -> Air_Coils_SML_NEOSID:Neosid_Air-Coil_SML_6turn_HAM0631A
- gave numbers to parts that had none: 1
Connections:
- no-connect marks 0 -> 16
